Commit message: modified code

File: urdf/ms616.urdf (robot description, URDF)
Before this commit: robot ms616, 6 links, 5 joints
Links:
- added link caster_link_back, mass 0.05; collision sphere radius=0.0206; visual mesh filename=package://ms616/meshes/caster.stl scale=0.001 0.001 0.001
- added link imu_link, mass 0.01; collision box size=0.02 0.02 0.01; visual box size=0.02 0.02 0.01
- link base_link: mass 2.0 -> 20.0
Joints:
- added joint caster_joint_back: type fixed, parent base_link, child caster_link_back, origin xyz=0.055 0 -0.0042 rpy=-1.5707 0 0
- added joint imu_joint: type fixed, parent base_link, child imu_link, origin xyz=0 0 0.05 rpy=0 0 0
- joint caster_joint: origin xyz=-0.055 0 -0.005 rpy=-1.5707 0 0 -> xyz=-0.055 0 -0.0042 rpy=-1.5707 0 0
